Commit message: update webserver, backup sh file

File: src/robot_model_pkg/urdf/robot_core.xacro (robot description, xacro)
@@ -3,6 +3,6 @@
 <!-- Here we define the model parameters -->
     <!-- Geometry -->
-    <xacro:property name="base_link_width" value="0.4"/>
-    <xacro:property name="base_link_length" value="0.4"/>
+    <xacro:property name="base_link_width" value="0.35"/>
+    <xacro:property name="base_link_length" value="0.35"/>
     <xacro:property name="base_link_height" value="0.05"/>
     <xacro:property name="wheel_link_length" value="0.03"/>
